File: Schematic/Lawo 28x16 with LED Matrix Components.sch (KiCad schematic (older format))
At the start: 10 parts, among them IC1 FP2800A, J1 Conn_02x25_Counter_Clockwise, J2 Conn_02x25_Counter_Clockwise, J3 Conn_01x02, J4 Conn_01x02

Commit message: Some open todos resolved and orientation/placing of the footprints changed
resolved todos:
- review mapping of the enable pins (remeasured on the physical hardware, newly labeled in the schematic, ...)
- review which connector receives the incoming signals and which goes to the next module

additional changes:
- connectors rotated and flipped to viewed from bottom side
- IC rotated
- connectors and IC rearranged to match their placement as seen from the front side to ease tracing and testing
- additional notes placed to highlight component placement, usage and things to take care about
Connections:
- net labels added: ENABLE_B, ENABLE_C, ENABLE_D
- net labels removed: ENABLE_1, ENABLE_2, ENABLE_3, ENABLE_4
- wire segments 189 -> 182
Other:
- note added: "Component mounted on the back side and shown here as accessible from the front.\nPositioned on the left edge. Incoming data signal from controller or previous matrix."
- note added: "Component mounted on the back side and shown here as accessible from the front.\nPositioned on the right edge. Outgoing data signal with slightly changed \nenable pins to allow cascading/daisy-chaining.\n"
- note added: "Connector (cascading)"
- note added: "Connector (incoming)"
- note added: "Please note:\nDo not cascade/chain more than 4 matrix modules to avoid overloading the driver ICs. \nThe mapping of the activation pins in the fifth matrix returns to the same assignment \nas for the first one, which would cause that two or more dots will be be triggered \nsimultaneously. This could draw or sink more power than the driver IC is able to handle."
- note added: "ToDo:\n- review naming of the enable pins\n (maybe align with ones of Lawo 28x13)\n- add more rating details about the mounted capacitors, \n resistors and LEDs\n- add schematic for the LED wiring\n- measure LED voltage level and fix schematic"
- note removed: "Connector"
- note removed: "ToDo:\n- review mapping of the enable pins\n- review naming of the enable pins (mayb align with ones of Lawo 28x13)\n- review which connector receives the incomming signals and which goes to the next module\n- add more rating details about the mounted capacitors, resistors and LEDs\n- add schematic for the LED wiring\n- measure LED voltage level and fix schematic"

Commit message: Again updates to the enable pins assignment, switch of the connectors and their usage (incoming <> cascading).
Parts:
- renumbered J2 to J1, J1 to J2
Other:
- note added: "Component mounted on the back side and shown here as accessible from the front.\nPositioned on the left edge. Outgoing data signal with slightly changed enable pins \nto allow cascading/daisy-chaining."
- note added: "Component mounted on the back side and shown here as accessible from the front.\nPositioned on the right edge. Incoming data signal from controller or previous matrix."
- note added: "ToDo:\n- review naming of the enable pins\n (maybe align with ones of Lawo 28x13)\n- add more rating details about the mounted LEDs \n and their resistor networks\n- add schematic for the LED wiring\n- measure LED voltage level and fix schematic"
- note removed: "Component mounted on the back side and shown here as accessible from the front.\nPositioned on the left edge. Incoming data signal from controller or previous matrix."
- note removed: "Component mounted on the back side and shown here as accessible from the front.\nPositioned on the right edge. Outgoing data signal with slightly changed \nenable pins to allow cascading/daisy-chaining.\n"
- note removed: "ToDo:\n- review naming of the enable pins\n (maybe align with ones of Lawo 28x13)\n- add more rating details about the mounted capacitors, \n resistors and LEDs\n- add schematic for the LED wiring\n- measure LED voltage level and fix schematic"
